File: ADE9000_Breakout.kicad_sch (KiCad schematic)
At the start: 56 parts, among them J1 Digital breadboard, J2 Voltage terminal, J3 Voltage terminal, J4 Voltage terminal, U1 ADE9000, Y1 24.576MHz

Commit message: Add 12 VAC voltage input support
Parts:
- added R21, R22, R23, R24, R25, R26: 100k, Resistor_SMD:R_0402_1005Metric, symbol Device:R
- added R27, R28, R29, R30, R31, R32: 2.49k, Resistor_SMD:R_0402_1005Metric, symbol Device:R
- J2, J3, J4: footprint TerminalBlock_4Ucon:TerminalBlock_4Ucon_1x02_P3.50mm_Horizontal -> ADE9000-Local:TerminalBlock_4Ucon_1x02_P3.50mm_Horizontal_ADE9000
Connections:
- net CLKIN: now also R27.2, R28.2, R29.2, R30.2, R31.2, R32.2
- net VAN_J: now also R22.1; no longer R10.1
- net VAP_J: now also R21.1; no longer R11.1
- net VBN_J: now also R24.1; no longer R12.1
- net VBP_J: now also R23.1; no longer R13.1
- net VCN_J: now also R26.1; no longer R14.1
- net VCP_J: now also R25.1; no longer R15.1
- new net VAN_DIV: R10.1, R22.2, R28.1
- new net VAP_DIV: R11.1, R21.2, R27.1
- new net VBN_DIV: R12.1, R24.2, R30.1
- new net VBP_DIV: R13.1, R23.2, R29.1
- new net VCN_DIV: R14.1, R26.2, R32.1
- new net VCP_DIV: R15.1, R25.2, R31.1
Other:
- moved on the sheet: C20, C22, C23, C24, C25, R10, R12, R13, R14, R15

Commit message: Use 0603 passives for hand assembly
Parts:
- C10, C9: footprint Capacitor_SMD:C_0402_1005Metric -> Capacitor_SMD:C_0603_1608Metric; DigiKey https://www.digikey.com/en/products/result?keywords=GRM1555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 -> https://www.digikey.com/en/products/result?keywords=GRM1885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; MPN GRM1555C1H160JA01D -> GRM1885C1H160JA01D; Mouser https://www.mouser.com/c/?q=GRM1555C1H160JA01D -> https://www.mouser.com/c/?q=GRM1885C1H160JA01D
- C11: footprint Capacitor_SMD:C_0402_1005Metric -> Capacitor_SMD:C_0603_1608Metric; DigiKey https://www.digikey.com/en/products/result?keywords=GRM155R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 -> https://www.digikey.com/en/products/result?keywords=GRM188R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; MPN GRM155R61A105KE15D -> GRM188R61A105KA61D; Mouser https://www.mouser.com/c/?q=GRM155R61A105KE15D -> https://www.mouser.com/c/?q=GRM188R61A105KA61D
- C12, C13, C14, C15, C16, C17, C18, C19, C20, C21, C22, C23, C24, C25: footprint Capacitor_SMD:C_0402_1005Metric -> Capacitor_SMD:C_0603_1608Metric; DigiKey https://www.digikey.com/en/products/result?keywords=GRM155R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 -> https://www.digikey.com/en/products/result?keywords=GRM188R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; MPN GRM155R71H223KA12D -> GRM188R71H223KA01D; Mouser https://www.mouser.com/c/?q=GRM155R71H223KA12D -> https://www.mouser.com/c/?q=GRM188R71H223KA01D
- C2, C4, C6, C8: footprint Capacitor_SMD:C_0402_1005Metric -> Capacitor_SMD:C_0603_1608Metric; DigiKey https://www.digikey.com/en/products/result?keywords=GRM155R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 -> https://www.digikey.com/en/products/result?keywords=GRM188R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; MPN GRM155R71A104KA01D -> GRM188R71A104KA61D; Mouser https://www.mouser.com/c/?q=GRM155R71A104KA01D -> https://www.mouser.com/c/?q=GRM188R71A104KA61D
- R1: footprint Resistor_SMD:R_0402_1005Metric -> Resistor_SMD:R_0603_1608Metric; DigiKey https://www.digikey.com/en/products/result?keywords=RC0402F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 -> https://www.digikey.com/en/products/result?keywords=RC0603F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; MPN RC0402FR-0710KL -> RC0603FR-0710KL; Mouser https://www.mouser.com/c/?q=RC0402FR-0710KL -> https://www.mouser.com/c/?q=RC0603FR-0710KL
- R10, R11, R12, R13, R14, R15, R16, R2, R3, R4, R5, R6, R7, R8, R9: footprint Resistor_SMD:R_0402_1005Metric -> Resistor_SMD:R_0603_1608Metric; DigiKey https://www.digikey.com/en/products/result?keywords=RC0402F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 -> https://www.digikey.com/en/products/result?keywords=RC0603F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; MPN RC0402FR-071KL -> RC0603FR-071KL; Mouser https://www.mouser.com/c/?q=RC0402FR-071KL -> https://www.mouser.com/c/?q=RC0603FR-071KL
- R17, R18, R19, R20: footprint Resistor_SMD:R_0402_1005Metric -> Resistor_SMD:R_0603_1608Metric; DigiKey https://www.digikey.com/en/products/result?keywords=RC0402F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 -> https://www.digikey.com/en/products/result?keywords=RC0603F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; MPN RC0402FR-072R4L -> RC0603FR-072R4L; Mouser https://www.mouser.com/c/?q=RC0402FR-072R4L -> https://www.mouser.com/c/?q=RC0603FR-072R4L
- R21, R22, R23, R24, R25, R26: footprint Resistor_SMD:R_0402_1005Metric -> Resistor_SMD:R_0603_1608Metric; DigiKey https://www.digikey.com/en/products/result?keywords=RC0402F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 -> https://www.digikey.com/en/products/result?keywords=RC0603F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; MPN RC0402FR-07100KL -> RC0603FR-07100KL; Mouser https://www.mouser.com/c/?q=RC0402FR-07100KL -> https://www.mouser.com/c/?q=RC0603FR-07100KL
- R27, R28, R29, R30, R31, R32: footprint Resistor_SMD:R_0402_1005Metric -> Resistor_SMD:R_0603_1608Metric; DigiKey https://www.digikey.com/en/products/result?keywords=RC0402F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 -> https://www.digikey.com/en/products/result?keywords=RC0603F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; MPN RC0402FR-072K49L -> RC0603FR-072K49L; Mouser https://www.mouser.com/c/?q=RC0402FR-072K49L -> https://www.mouser.com/c/?q=RC0603FR-072K49L
