File: ADE9000_Breakout.kicad_sch (KiCad schematic)
At the start: 68 parts, among them J1 Digital breadboard, J2 Voltage terminal, J3 Voltage terminal, J4 Voltage terminal, U1 ADE9000, Y1 24.576MHz

Commit message: Add selectable ADE9000 power modes
Add ATM-style PM0/PM1 solder bridges, regenerate the routed board and BOM, and publish populated isometric renders in the README.\n\nCo-authored-by: Copilot <223556219+Copilot@users.noreply.github.com>
Parts:
- added JP1: PM0 mode, ADE9000-Local:ModeBridge_3Pad, symbol Jumper:SolderJumper_3_Open
- added JP2: PM1 mode, ADE9000-Local:ModeBridge_3Pad, symbol Jumper:SolderJumper_3_Open
- C2, C4, C6, C8: DigiKey https://www.digikey.com/en/products/result?keywords=GRM188R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 -> https://www.digikey.com.au/en/products/detail/yageo/CC0603K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; MPN GRM188R71A104KA61D -> CC0603KPX7R0BB104; Manufacturer Murata -> YAGEO; Mouser https://www.mouser.com/c/?q=GRM188R71A104KA61D -> https://www.mouser.com/c/?q=CC0603KPX7R0BB104
Connections:
- net +3V3: now also JP1.1 (A), JP2.1 (A)
- net CLKIN: now also JP1.3 (B), JP2.3 (B); no longer U1.4 (PM0), U1.5 (PM1)
- new net PM0: JP1.2 (C), U1.4 (PM0)
- new net PM1: JP2.2 (C), U1.5 (PM1)
